Commit message: Add depth camera plugin successfully

File: simulator/models/urdf/depth_camera.xacro (robot description, xacro)
@@ -27,4 +27,5 @@
                 </geometry>
             </collision>
+        </link>
             <gazebo reference="depth_camera">
                 <sensor name="camera" type="depth">
@@ -68,5 +69,4 @@
                 </sensor>
             </gazebo>
-        </link>
     </xacro:macro>
 </robot>
